File: Inverter.kicad_sch (KiCad schematic)
At the start: 16 parts, among them J3 2 way net tie junction, Q1 ${MANUFACTURER PART NUMBER}, Q2 ${MANUFACTURER PART NUMBER}, U6 ${MANUFACTURER PART NUMBER}, U7 ${MANUFACTURER PART NUMBER}

Commit message: rename project
Other:
- title: EPC_25 -> KA30GAN
Changed lines of the file:
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@@
   (paper "A4")
   (title_block
-    (title "EPC_25")
+    (title "KA30GAN")
     (rev "1.0")
     (company "IPM Group ©")
@@
     (pin "1")
     (instances
-      (project "EPC_25"
+      (project "ka30gan"
         (path "/2fa95553-e4bc-4555-b37d-4bed2a7cfe1b/a4711c07-37a1-4f3c-8856-aaf7e93600b6"
           (reference "J3") (unit 1)
@@
     (pin "")
     (instances
-      (project "EPC_25"
+      (project "ka30gan"
         (path "/2fa95553-e4bc-4555-b37d-4bed2a7cfe1b/a4711c07-37a1-4f3c-8856-aaf7e93600b6"
           (reference "#PWR044") (unit 1)
@@
     (pin "6")
     (instances
-      (project "EPC_25"
+      (project "ka30gan"
         (path "/2fa95553-e4bc-4555-b37d-4bed2a7cfe1b/a4711c07-37a1-4f3c-8856-aaf7e93600b6"
           (reference "U7") (unit 1)
@@
     (pin "2")
     (instances
-      (project "EPC_25"
+      (project "ka30gan"
         (path "/2fa95553-e4bc-4555-b37d-4bed2a7cfe1b/a4711c07-37a1-4f3c-8856-aaf7e93600b6"
           (reference "R17") (unit 1)
@@
     (pin "2")
     (instances
-      (project "EPC_25"
+      (project "ka30gan"
         (path "/2fa95553-e4bc-4555-b37d-4bed2a7cfe1b/a4711c07-37a1-4f3c-8856-aaf7e93600b6"
           (reference "C31") (unit 1)
@@
     (pin "")
     (instances
-      (project "EPC_25"
+      (project "ka30gan"
         (path "/2fa95553-e4bc-4555-b37d-4bed2a7cfe1b/a4711c07-37a1-4f3c-8856-aaf7e93600b6"
           (reference "#PWR046") (unit 1)
@@
     (pin "9")
     (instances
-      (project "EPC_25"
+      (project "ka30gan"
         (path "/2fa95553-e4bc-4555-b37d-4bed2a7cfe1b/a4711c07-37a1-4f3c-8856-aaf7e93600b6"
           (reference "Q2") (unit 1)
@@
     (pin "2")
     (instances
-      (project "EPC_25"
+      (project "ka30gan"
         (path "/2fa95553-e4bc-4555-b37d-4bed2a7cfe1b/a4711c07-37a1-4f3c-8856-aaf7e93600b6"
           (reference "C26") (unit 1)
@@
     (pin "")
     (instances
-      (project "EPC_25"
+      (project "ka30gan"
         (path "/2fa95553-e4bc-4555-b37d-4bed2a7cfe1b/a4711c07-37a1-4f3c-8856-aaf7e93600b6"
           (reference "#PWR042") (unit 1)
@@
     (pin "2")
     (instances
-      (project "EPC_25"
+      (project "ka30gan"
         (path "/2fa95553-e4bc-4555-b37d-4bed2a7cfe1b/a4711c07-37a1-4f3c-8856-aaf7e93600b6"
           (reference "C30") (unit 1)
@@
     (pin "2")
     (instances
-      (project "EPC_25"
+      (project "ka30gan"
         (path "/2fa95553-e4bc-4555-b37d-4bed2a7cfe1b/a4711c07-37a1-4f3c-8856-aaf7e93600b6"
           (reference "R16") (unit 1)
@@
     (pin "2")
     (instances
-      (project "EPC_25"
+      (project "ka30gan"
         (path "/2fa95553-e4bc-4555-b37d-4bed2a7cfe1b/a4711c07-37a1-4f3c-8856-aaf7e93600b6"
           (reference "C33") (unit 1)
@@
     (pin "")
     (instances
-      (project "EPC_25"
+      (project "ka30gan"
         (path "/2fa95553-e4bc-4555-b37d-4bed2a7cfe1b/a4711c07-37a1-4f3c-8856-aaf7e93600b6"
           (reference "#PWR045") (unit 1)
@@
     (pin "2")
     (instances
-      (project "EPC_25"
+      (project "ka30gan"
         (path "/2fa95553-e4bc-4555-b37d-4bed2a7cfe1b/a4711c07-37a1-4f3c-8856-aaf7e93600b6"
           (reference "C34") (unit 1)
@@
     (pin "D4")
     (instances
-      (project "EPC_25"
+      (project "ka30gan"
         (path "/2fa95553-e4bc-4555-b37d-4bed2a7cfe1b/a4711c07-37a1-4f3c-8856-aaf7e93600b6"
           (reference "U6") (unit 1)
@@
     (pin "2")
     (instances
-      (project "EPC_25"
+      (project "ka30gan"
         (path "/2fa95553-e4bc-4555-b37d-4bed2a7cfe1b/a4711c07-37a1-4f3c-8856-aaf7e93600b6"
           (reference "C29") (unit 1)
@@
     (pin "")
     (instances
-      (project "EPC_25"
+      (project "ka30gan"
         (path "/2fa95553-e4bc-4555-b37d-4bed2a7cfe1b/a4711c07-37a1-4f3c-8856-aaf7e93600b6"
           (reference "#PWR047") (unit 1)
@@
     (pin "")
     (instances
-      (project "EPC_25"
+      (project "ka30gan"
         (path "/2fa95553-e4bc-4555-b37d-4bed2a7cfe1b/a4711c07-37a1-4f3c-8856-aaf7e93600b6"
           (reference "#PWR048") (unit 1)
@@
     (pin "9")
     (instances
-      (project "EPC_25"
+      (project "ka30gan"
         (path "/2fa95553-e4bc-4555-b37d-4bed2a7cfe1b/a4711c07-37a1-4f3c-8856-aaf7e93600b6"
           (reference "Q1") (unit 1)
@@
     (pin "")
     (instances
-      (project "EPC_25"
+      (project "ka30gan"
         (path "/2fa95553-e4bc-4555-b37d-4bed2a7cfe1b/a4711c07-37a1-4f3c-8856-aaf7e93600b6"
           (reference "#PWR043") (unit 1)
@@
     (pin "")
     (instances
-      (project "EPC_25"
+      (project "ka30gan"
         (path "/2fa95553-e4bc-4555-b37d-4bed2a7cfe1b/a4711c07-37a1-4f3c-8856-aaf7e93600b6"
           (reference "#PWR041") (unit 1)
@@
     (pin "2")
     (instances
-      (project "EPC_25"
+      (project "ka30gan"
         (path "/2fa95553-e4bc-4555-b37d-4bed2a7cfe1b/a4711c07-37a1-4f3c-8856-aaf7e93600b6"
           (reference "C32") (unit 1)
@@
     (pin "2")
     (instances
-      (project "EPC_25"
+      (project "ka30gan"
         (path "/2fa95553-e4bc-4555-b37d-4bed2a7cfe1b/a4711c07-37a1-4f3c-8856-aaf7e93600b6"
           (reference "C27") (unit 1)
@@
     (pin "2")
     (instances
-      (project "EPC_25"
+      (project "ka30gan"
         (path "/2fa95553-e4bc-4555-b37d-4bed2a7cfe1b/a4711c07-37a1-4f3c-8856-aaf7e93600b6"
           (reference "C28") (unit 1)

Commit message: edit sym
Parts:
- C26: symbol EPC_25-altium-import:root_1_Capacitor -> ka30gan:root_1_Capacitor; ALTIUM_VALUE 4.7uF -> (none)
- C27, C29, C30, C32, C33: symbol EPC_25-altium-import:root_1_Capacitor -> ka30gan:root_1_Capacitor; ALTIUM_VALUE 1uF -> (none)
- C28: symbol EPC_25-altium-import:root_0_Capacitor -> ka30gan:root_0_Capacitor; ALTIUM_VALUE 0.1uF -> (none)
- C31, C34: symbol EPC_25-altium-import:root_1_Capacitor -> ka30gan:root_1_Capacitor; ALTIUM_VALUE 0.1uF -> (none)
- J3: symbol EPC_25-altium-import:root_0_1way -> ka30gan:root_0_1way
- Q1, Q2: symbol EPC_25-altium-import:root_0_MOSFET EPC2021 -> ka30gan:root_0_MOSFET EPC2021
- R16: symbol EPC_25-altium-import:root_1_Resistor -> ka30gan:root_1_Resistor; ALTIUM_VALUE 47000 -> (none)
- R17: symbol EPC_25-altium-import:root_1_Resistor -> ka30gan:root_1_Resistor; ALTIUM_VALUE 4990 -> (none)
- U6: symbol EPC_25-altium-import:root_0_LMG1205YFXR -> ka30gan:root_0_LMG1205YFXR
- U7: symbol EPC_25-altium-import:root_0_ACS711KEXLT-31AB-T -> ka30gan:root_0_ACS711KEXLT-31AB-T
