File: Power.kicad_sch (KiCad schematic)
At the start: 15 parts, among them J1 2 way net tie junction, J2 2 way net tie junction, T11 Test_Point_L, T12 Test_Point_L, U3 ${MANUFACTURER PART NUMBER}, U4 ${MANUFACTURER PART NUMBER}

Commit message: rename project
Other:
- title: EPC_25 -> KA30GAN
Changed lines of the file:
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@@
   (paper "A4")
   (title_block
-    (title "EPC_25")
+    (title "KA30GAN")
     (rev "1.0")
     (company "IPM Group ©")
@@
     (pin "")
     (instances
-      (project "EPC_25"
+      (project "ka30gan"
         (path "/2fa95553-e4bc-4555-b37d-4bed2a7cfe1b/53a0bca7-8d4b-442b-ade3-5bde439fe9e9"
           (reference "#PWR027") (unit 1)
@@
     (pin "2")
     (instances
-      (project "EPC_25"
+      (project "ka30gan"
         (path "/2fa95553-e4bc-4555-b37d-4bed2a7cfe1b/53a0bca7-8d4b-442b-ade3-5bde439fe9e9"
           (reference "R13") (unit 1)
@@
     (pin "")
     (instances
-      (project "EPC_25"
+      (project "ka30gan"
         (path "/2fa95553-e4bc-4555-b37d-4bed2a7cfe1b/53a0bca7-8d4b-442b-ade3-5bde439fe9e9"
           (reference "#PWR030") (unit 1)
@@
     (pin "2")
     (instances
-      (project "EPC_25"
+      (project "ka30gan"
         (path "/2fa95553-e4bc-4555-b37d-4bed2a7cfe1b/53a0bca7-8d4b-442b-ade3-5bde439fe9e9"
           (reference "R14") (unit 1)
@@
     (pin "1")
     (instances
-      (project "EPC_25"
+      (project "ka30gan"
         (path "/2fa95553-e4bc-4555-b37d-4bed2a7cfe1b/53a0bca7-8d4b-442b-ade3-5bde439fe9e9"
           (reference "J2") (unit 1)
@@
     (pin "2")
     (instances
-      (project "EPC_25"
+      (project "ka30gan"
         (path "/2fa95553-e4bc-4555-b37d-4bed2a7cfe1b/53a0bca7-8d4b-442b-ade3-5bde439fe9e9"
           (reference "C22") (unit 1)
@@
     (pin "2")
     (instances
-      (project "EPC_25"
+      (project "ka30gan"
         (path "/2fa95553-e4bc-4555-b37d-4bed2a7cfe1b/53a0bca7-8d4b-442b-ade3-5bde439fe9e9"
           (reference "D4") (unit 1)
@@
     (pin "")
     (instances
-      (project "EPC_25"
+      (project "ka30gan"
         (path "/2fa95553-e4bc-4555-b37d-4bed2a7cfe1b/53a0bca7-8d4b-442b-ade3-5bde439fe9e9"
           (reference "#PWR031") (unit 1)
@@
     (pin "7")
     (instances
-      (project "EPC_25"
+      (project "ka30gan"
         (path "/2fa95553-e4bc-4555-b37d-4bed2a7cfe1b/53a0bca7-8d4b-442b-ade3-5bde439fe9e9"
           (reference "U3") (unit 1)
@@
     (pin "2")
     (instances
-      (project "EPC_25"
+      (project "ka30gan"
         (path "/2fa95553-e4bc-4555-b37d-4bed2a7cfe1b/53a0bca7-8d4b-442b-ade3-5bde439fe9e9"
           (reference "C21") (unit 1)
@@
     (pin "1")
     (instances
-      (project "EPC_25"
+      (project "ka30gan"
         (path "/2fa95553-e4bc-4555-b37d-4bed2a7cfe1b/53a0bca7-8d4b-442b-ade3-5bde439fe9e9"
           (reference "T12") (unit 1)
@@
     (pin "")
     (instances
-      (project "EPC_25"
+      (project "ka30gan"
         (path "/2fa95553-e4bc-4555-b37d-4bed2a7cfe1b/53a0bca7-8d4b-442b-ade3-5bde439fe9e9"
           (reference "#PWR021") (unit 1)
@@
     (pin "")
     (instances
-      (project "EPC_25"
+      (project "ka30gan"
         (path "/2fa95553-e4bc-4555-b37d-4bed2a7cfe1b/53a0bca7-8d4b-442b-ade3-5bde439fe9e9"
           (reference "#PWR025") (unit 1)
@@
     (pin "1")
     (instances
-      (project "EPC_25"
+      (project "ka30gan"
         (path "/2fa95553-e4bc-4555-b37d-4bed2a7cfe1b/53a0bca7-8d4b-442b-ade3-5bde439fe9e9"
           (reference "T11") (unit 1)
@@
     (pin "")
     (instances
-      (project "EPC_25"
+      (project "ka30gan"
         (path "/2fa95553-e4bc-4555-b37d-4bed2a7cfe1b/53a0bca7-8d4b-442b-ade3-5bde439fe9e9"
           (reference "#PWR022") (unit 1)
@@
     (pin "")
     (instances
-      (project "EPC_25"
+      (project "ka30gan"
         (path "/2fa95553-e4bc-4555-b37d-4bed2a7cfe1b/53a0bca7-8d4b-442b-ade3-5bde439fe9e9"
           (reference "#PWR023") (unit 1)
@@
     (pin "2")
     (instances
-      (project "EPC_25"
+      (project "ka30gan"
         (path "/2fa95553-e4bc-4555-b37d-4bed2a7cfe1b/53a0bca7-8d4b-442b-ade3-5bde439fe9e9"
           (reference "C19") (unit 1)
@@
     (pin "")
     (instances
-      (project "EPC_25"
+      (project "ka30gan"
         (path "/2fa95553-e4bc-4555-b37d-4bed2a7cfe1b/53a0bca7-8d4b-442b-ade3-5bde439fe9e9"
           (reference "#PWR026") (unit 1)
@@
     (pin "2")
     (instances
-      (project "EPC_25"
+      (project "ka30gan"
         (path "/2fa95553-e4bc-4555-b37d-4bed2a7cfe1b/53a0bca7-8d4b-442b-ade3-5bde439fe9e9"
           (reference "C23") (unit 1)
@@
     (pin "")
     (instances
-      (project "EPC_25"
+      (project "ka30gan"
         (path "/2fa95553-e4bc-4555-b37d-4bed2a7cfe1b/53a0bca7-8d4b-442b-ade3-5bde439fe9e9"
           (reference "#PWR024") (unit 1)
@@
     (pin "2")
     (instances
-      (project "EPC_25"
+      (project "ka30gan"
         (path "/2fa95553-e4bc-4555-b37d-4bed2a7cfe1b/53a0bca7-8d4b-442b-ade3-5bde439fe9e9"
           (reference "C20") (unit 1)
@@
     (pin "")
     (instances
-      (project "EPC_25"
+      (project "ka30gan"
         (path "/2fa95553-e4bc-4555-b37d-4bed2a7cfe1b/53a0bca7-8d4b-442b-ade3-5bde439fe9e9"
           (reference "#PWR028") (unit 1)
@@
     (pin "7")
     (instances
-      (project "EPC_25"
+      (project "ka30gan"
         (path "/2fa95553-e4bc-4555-b37d-4bed2a7cfe1b/53a0bca7-8d4b-442b-ade3-5bde439fe9e9"
           (reference "U4") (unit 1)
@@
     (pin "1")
     (instances
-      (project "EPC_25"
+      (project "ka30gan"
         (path "/2fa95553-e4bc-4555-b37d-4bed2a7cfe1b/53a0bca7-8d4b-442b-ade3-5bde439fe9e9"
           (reference "J1") (unit 1)
@@
     (pin "2")
     (instances
-      (project "EPC_25"
+      (project "ka30gan"
         (path "/2fa95553-e4bc-4555-b37d-4bed2a7cfe1b/53a0bca7-8d4b-442b-ade3-5bde439fe9e9"
           (reference "R12") (unit 1)
@@
     (pin "")
     (instances
-      (project "EPC_25"
+      (project "ka30gan"
         (path "/2fa95553-e4bc-4555-b37d-4bed2a7cfe1b/53a0bca7-8d4b-442b-ade3-5bde439fe9e9"
           (reference "#PWR029") (unit 1)

Commit message: edit sym
Parts:
- C19: symbol EPC_25-altium-import:root_1_Capacitor -> ka30gan:root_1_Capacitor; ALTIUM_VALUE 10uF -> (none)
- C20, C22: symbol EPC_25-altium-import:root_1_Capacitor -> ka30gan:root_1_Capacitor; ALTIUM_VALUE 2.2uF -> (none)
- C21: symbol EPC_25-altium-import:root_1_Capacitor -> ka30gan:root_1_Capacitor; ALTIUM_VALUE 0.01uF -> (none)
- C23: symbol EPC_25-altium-import:root_1_Capacitor -> ka30gan:root_1_Capacitor; ALTIUM_VALUE 47uF -> (none)
- D4: symbol EPC_25-altium-import:root_3_LED Green 0402 -> ka30gan:root_3_LED Green 0402; AUTHOR AB -> (none)
- J1, J2: symbol EPC_25-altium-import:root_0_1way -> ka30gan:root_0_1way
- R12: symbol EPC_25-altium-import:root_1_Resistor -> ka30gan:root_1_Resistor; ALTIUM_VALUE 24300 -> (none)
- R13: symbol EPC_25-altium-import:root_0_Resistor -> ka30gan:root_0_Resistor; ALTIUM_VALUE 100000 -> (none)
- R14: symbol EPC_25-altium-import:root_1_Resistor -> ka30gan:root_1_Resistor; ALTIUM_VALUE 330 -> (none)
- T11, T12: symbol EPC_25-altium-import:root_0_Test_Point_L -> ka30gan:root_0_Test_Point_L
- U3: symbol EPC_25-altium-import:root_0_LMZM23601SILT -> ka30gan:root_0_LMZM23601SILT
- U4: symbol EPC_25-altium-import:root_0_TPS73533DRVR -> ka30gan:root_0_TPS73533DRVR
Connections:
- no-connect marks 0 -> 1
Other:
- moved on the sheet: C20, C21, C22, D4, R14, T11, U4

Commit message: fix DRC
Changed lines of the file:
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@@
   (junction (at 163.83 81.28) (diameter 0) (color 0 0 0 0)
+  )
+  (junction (at 123.19 76.2) (diameter 0) (color 0 0 0 0)
   )
   (junction (at 173.99 76.2) (diameter 0) (color 0 0 0 0)
@@
   (wire (pts (xy 123.19 128.27) (xy 123.19 125.73))
     (stroke (width 0.254) (type default))
+  )
+  (wire (pts (xy 179.07 88.9) (xy 191.77 88.9))
+    (stroke (width 0) (type default))
   )
   (wire (pts (xy 179.07 88.9) (xy 163.83 88.9))
@@
         )
       )
+    )
+  )
+  (symbol (lib_id "power:PWR_FLAG") (at 191.77 88.9 0) (unit 1)
+    (in_bom yes) (on_board yes) (dnp no) (fields_autoplaced)
+    (property "Reference" "#FLG01" (at 191.77 86.995 0)
+      (effects (font (size 1.27 1.27)) hide)
+    )
+    (property "Value" "PWR_FLAG" (at 191.77 83.82 0)
+      (effects (font (size 1.27 1.27)))
+    )
+    (property "Footprint" "" (at 191.77 88.9 0)
+      (effects (font (size 1.27 1.27)) hide)
+    )
+    (property "Datasheet" "~" (at 191.77 88.9 0)
+      (effects (font (size 1.27 1.27)) hide)
+    )
+    (pin "1")
+    (instances
+      (project "ka30gan"
+        (path "/2fa95553-e4bc-4555-b37d-4bed2a7cfe1b"
+          (reference "#FLG01") (unit 1)
+        )
+        (path "/2fa95553-e4bc-4555-b37d-4bed2a7cfe1b/53a0bca7-8d4b-442b-ade3-5bde439fe9e9"
+          (reference "#FLG06") (unit 1)
+        )
+      )
+    )
+  )
+  (symbol (lib_id "power:PWR_FLAG") (at 123.19 76.2 0) (unit 1)
+    (in_bom yes) (on_board yes) (dnp no) (fields_autoplaced)
+    (property "Reference" "#FLG01" (at 123.19 74.295 0)
+      (effects (font (size 1.27 1.27)) hide)
+    )
+    (property "Value" "PWR_FLAG" (at 123.19 71.12 0)
+      (effects (font (size 1.27 1.27)))
+    )
+    (property "Footprint" "" (at 123.19 76.2 0)
+      (effects (font (size 1.27 1.27)) hide)
+    )
+    (property "Datasheet" "~" (at 123.19 76.2 0)
+      (effects (font (size 1.27 1.27)) hide)
+    )
+    (pin "1")
+    (instances
+      (project "ka30gan"
+        (path "/2fa95553-e4bc-4555-b37d-4bed2a7cfe1b"
+          (reference "#FLG01") (unit 1)
+        )
+        (path "/2fa95553-e4bc-4555-b37d-4bed2a7cfe1b/53a0bca7-8d4b-442b-ade3-5bde439fe9e9"
+          (reference "#FLG03") (unit 1)
+        )
+      )
