File: ka30gan.kicad_sch (KiCad schematic)
At the start: 52 parts, among them T1 Test_Point_L, T10 Test_Point_L, T2 Test_Point_L, T3 Test_Point_L, T4 Test_Point_L, T5 Test_Point_L, T6 Test_Point_L, T7 Test_Point_L, T8 Test_Point_L, T9 Test_Point_L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

Commit message: edit sym
Parts:
- C1, C16, C17, C18: symbol EPC_25-altium-import:root_1_Capacitor -> ka30gan:root_1_Capacitor; ALTIUM_VALUE 0.1uF -> (none)
- C10, C11, C12, C5, C6, C7: symbol EPC_25-altium-import:root_0_Capacitor -> ka30gan:root_0_Capacitor; ALTIUM_VALUE 2.2uF -> (none)
- C13, C14, C15, C2, C3, C4, C8, C9: symbol EPC_25-altium-import:root_1_Capacitor -> ka30gan:root_1_Capacitor; ALTIUM_VALUE 2.2uF -> (none)
- D1: symbol EPC_25-altium-import:root_3_LED Red 0402 -> ka30gan:root_3_LED Red 0402; AUTHOR CERN DEM JLC -> (none)
- D2: symbol EPC_25-altium-import:root_0_ESD TPD4E05U06QDQARQ1 -> ka30gan:root_0_ESD TPD4E05U06QDQARQ1; AUTHOR AB -> (none)
- D3: symbol EPC_25-altium-import:root_3_LED Blue 0402 -> ka30gan:root_3_LED Blue 0402; AUTHOR AB -> (none)
- FID1, FID2, FID3, FID4, FID5, FID6: symbol EPC_25-altium-import:root_0_Fiducial -> ka30gan:root_0_Fiducial
- L1: symbol EPC_25-altium-import:root_0_L BKP1005HS221 -> ka30gan:root_0_L BKP1005HS221; ALTIUM_VALUE 220 ohm -> (none)
- L2: symbol EPC_25-altium-import:root_0_L BLM15PD600SN1D -> ka30gan:root_0_L BLM15PD600SN1D; ALTIUM_VALUE 60 ohm -> (none)
- R1, R7: symbol EPC_25-altium-import:root_1_Resistor -> ka30gan:root_1_Resistor; ALTIUM_VALUE 10000 -> (none)
- R10, R4, R5: symbol EPC_25-altium-import:root_1_Resistor -> ka30gan:root_1_Resistor; ALTIUM_VALUE 4990 -> (none)
- R11, R8: symbol EPC_25-altium-import:root_1_Resistor -> ka30gan:root_1_Resistor; ALTIUM_VALUE 330 -> (none)
- R2, R3, R6: symbol EPC_25-altium-import:root_1_Resistor -> ka30gan:root_1_Resistor; ALTIUM_VALUE 2200 -> (none)
- R9: symbol EPC_25-altium-import:root_1_Resistor -> ka30gan:root_1_Resistor; ALTIUM_VALUE 47000 -> (none)
- T1, T2, T3: symbol EPC_25-altium-import:root_0_Test_Point_L -> ka30gan:root_0_Test_Point_L
- T10, T4, T5, T6, T7, T8, T9: symbol EPC_25-altium-import:root_0_mirrored_Test_Point_L -> ka30gan:root_0_mirrored_Test_Point_L
- U1: symbol EPC_25-altium-import:root_0_TMS320F28062FPNT -> ka30gan:root_0_TMS320F28062FPNT
- U2: symbol EPC_25-altium-import:root_0_M24C16-FMH6TG -> ka30gan:root_0_M24C16-FMH6TG
Connections:
- no-connect marks 3 -> 28
Other:
- moved on the sheet: C2, C3, L1, L2

Commit message: fix DRC
Changed lines of the file:
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@@
   (junction (at 62.23 128.27) (diameter 0) (color 0 0 0 0)
   )
+  (junction (at 68.58 92.71) (diameter 0) (color 0 0 0 0)
+  )
   (junction (at 113.03 125.73) (diameter 0) (color 0 0 0 0)
   )
@@
     (stroke (width 0.254) (type default))
   )
-  (wire (pts (xy 46.99 92.71) (xy 77.47 92.71))
+  (wire (pts (xy 46.99 92.71) (xy 68.58 92.71))
     (stroke (width 0.254) (type default))
   )
@@
     (stroke (width 0.254) (type default))
   )
+  (wire (pts (xy 68.58 92.71) (xy 77.47 92.71))
+    (stroke (width 0.254) (type default))
+  )
   (wire (pts (xy 52.07 115.57) (xy 57.15 115.57))
     (stroke (width 0.254) (type default))
@@
     )
   )
+  (symbol (lib_id "power:PWR_FLAG") (at 68.58 92.71 0) (unit 1)
+    (in_bom yes) (on_board yes) (dnp no) (fields_autoplaced)
+    (property "Reference" "#FLG01" (at 68.58 90.805 0)
+      (effects (font (size 1.27 1.27)) hide)
+    )
+    (property "Value" "PWR_FLAG" (at 68.58 87.63 0)
+      (effects (font (size 1.27 1.27)))
+    )
+    (property "Footprint" "" (at 68.58 92.71 0)
+      (effects (font (size 1.27 1.27)) hide)
+    )
+    (property "Datasheet" "~" (at 68.58 92.71 0)
+      (effects (font (size 1.27 1.27)) hide)
+    )
+    (pin "1")
+    (instances
+      (project "ka30gan"
+        (path "/2fa95553-e4bc-4555-b37d-4bed2a7cfe1b"
+          (reference "#FLG01") (unit 1)
+        )
+      )
+    )
+  )
   (symbol (lib_id "ka30gan:root_1_Capacitor") (at 72.39 128.27 0) (unit 1)
     (in_bom yes) (on_board yes) (dnp no)
@@
         )
       )
+    )
+  )
+  (symbol (lib_id "power:PWR_FLAG") (at 46.99 115.57 0) (unit 1)
+    (in_bom yes) (on_board yes) (dnp no) (fields_autoplaced)
+    (property "Reference" "#FLG02" (at 46.99 113.665 0)
+      (effects (font (size 1.27 1.27)) hide)
+    )
+    (property "Value" "PWR_FLAG" (at 46.99 110.49 0)
+      (effects (font (size 1.27 1.27)))
+    )
+    (property "Footprint" "" (at 46.99 115.57 0)
+      (effects (font (size 1.27 1.27)) hide)
+    )
+    (property "Datasheet" "~" (at 46.99 115.57 0)
+      (effects (font (size 1.27 1.27)) hide)
+    )
+    (pin "1")
+    (instances
+      (project "ka30gan"
+        (path "/2fa95553-e4bc-4555-b37d-4bed2a7cfe1b"
+          (reference "#FLG02") (unit 1)
+        )
+      )
